File: optoinput.sch (KiCad schematic (older format))
At the start: 28 parts, among them P1 CONN_01X08, P2 CONN_01X08, P3 CONN_01X03, P6 CONN_01X02, U1 4N25, U2 4N25, U3 4N25, U4 4N25, U5 4N25, U6 4N25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

Commit message: schema mods
Parts:
- R1, R10, R11, R12, R2, R3, R4, R9: value R -> 1K
- R13, R14, R15, R16, R5, R6, R7, R8: value R -> 4.7K
Changed lines of the file:
@@
 P 1750 2850
 F 0 "R1" V 1830 2850 50  0000 C CNN
-F 1 "R" V 1750 2850 50  0000 C CNN
+F 1 "1K" V 1750 2850 50  0000 C CNN
 F 2 "Resistors_ThroughHole:Resistor_Horizontal_RM10mm" V 1680 2850 50  0001 C CNN
 F 3 "" H 1750 2850 50  0000 C CNN
@@
 P 2650 3350
 F 0 "R5" V 2730 3350 50  0000 C CNN
-F 1 "R" V 2650 3350 50  0000 C CNN
+F 1 "4.7K" V 2650 3350 50  0000 C CNN
 F 2 "Resistors_ThroughHole:Resistor_Horizontal_RM10mm" V 2580 3350 50  0001 C CNN
 F 3 "" H 2650 3350 50  0000 C CNN
@@
 P 3100 2850
 F 0 "R2" V 3180 2850 50  0000 C CNN
-F 1 "R" V 3100 2850 50  0000 C CNN
+F 1 "1K" V 3100 2850 50  0000 C CNN
 F 2 "Resistors_ThroughHole:Resistor_Horizontal_RM10mm" V 3030 2850 50  0001 C CNN
 F 3 "" H 3100 2850 50  0000 C CNN
@@
 P 4000 3350
 F 0 "R6" V 4080 3350 50  0000 C CNN
-F 1 "R" V 4000 3350 50  0000 C CNN
+F 1 "4.7K" V 4000 3350 50  0000 C CNN
 F 2 "Resistors_ThroughHole:Resistor_Horizontal_RM10mm" V 3930 3350 50  0001 C CNN
 F 3 "" H 4000 3350 50  0000 C CNN
@@
 P 4450 2850
 F 0 "R3" V 4530 2850 50  0000 C CNN
-F 1 "R" V 4450 2850 50  0000 C CNN
+F 1 "1K" V 4450 2850 50  0000 C CNN
 F 2 "Resistors_ThroughHole:Resistor_Horizontal_RM10mm" V 4380 2850 50  0001 C CNN
 F 3 "" H 4450 2850 50  0000 C CNN
@@
 P 5350 3350
 F 0 "R7" V 5430 3350 50  0000 C CNN
-F 1 "R" V 5350 3350 50  0000 C CNN
+F 1 "4.7K" V 5350 3350 50  0000 C CNN
 F 2 "Resistors_ThroughHole:Resistor_Horizontal_RM10mm" V 5280 3350 50  0001 C CNN
 F 3 "" H 5350 3350 50  0000 C CNN
@@
 P 5800 2850
 F 0 "R4" V 5880 2850 50  0000 C CNN
-F 1 "R" V 5800 2850 50  0000 C CNN
+F 1 "1K" V 5800 2850 50  0000 C CNN
 F 2 "Resistors_ThroughHole:Resistor_Horizontal_RM10mm" V 5730 2850 50  0001 C CNN
 F 3 "" H 5800 2850 50  0000 C CNN
@@
 P 6700 3350
 F 0 "R8" V 6780 3350 50  0000 C CNN
-F 1 "R" V 6700 3350 50  0000 C CNN
+F 1 "4.7K" V 6700 3350 50  0000 C CNN
 F 2 "Resistors_ThroughHole:Resistor_Horizontal_RM10mm" V 6630 3350 50  0001 C CNN
 F 3 "" H 6700 3350 50  0000 C CNN
@@
 P 1750 4350
 F 0 "R9" V 1830 4350 50  0000 C CNN
-F 1 "R" V 1750 4350 50  0000 C CNN
+F 1 "1K" V 1750 4350 50  0000 C CNN
 F 2 "Resistors_ThroughHole:Resistor_Horizontal_RM10mm" V 1680 4350 50  0001 C CNN
 F 3 "" H 1750 4350 50  0000 C CNN
@@
 P 2650 4850
 F 0 "R13" V 2730 4850 50  0000 C CNN
-F 1 "R" V 2650 4850 50  0000 C CNN
+F 1 "4.7K" V 2650 4850 50  0000 C CNN
 F 2 "Resistors_ThroughHole:Resistor_Horizontal_RM10mm" V 2580 4850 50  0001 C CNN
 F 3 "" H 2650 4850 50  0000 C CNN
@@
 P 3100 4350
 F 0 "R10" V 3180 4350 50  0000 C CNN
-F 1 "R" V 3100 4350 50  0000 C CNN
+F 1 "1K" V 3100 4350 50  0000 C CNN
 F 2 "Resistors_ThroughHole:Resistor_Horizontal_RM10mm" V 3030 4350 50  0001 C CNN
 F 3 "" H 3100 4350 50  0000 C CNN
@@
 P 4000 4850
 F 0 "R14" V 4080 4850 50  0000 C CNN
-F 1 "R" V 4000 4850 50  0000 C CNN
+F 1 "4.7K" V 4000 4850 50  0000 C CNN
 F 2 "Resistors_ThroughHole:Resistor_Horizontal_RM10mm" V 3930 4850 50  0001 C CNN
 F 3 "" H 4000 4850 50  0000 C CNN
@@
 P 4450 4350
 F 0 "R11" V 4530 4350 50  0000 C CNN
-F 1 "R" V 4450 4350 50  0000 C CNN
+F 1 "1K" V 4450 4350 50  0000 C CNN
 F 2 "Resistors_ThroughHole:Resistor_Horizontal_RM10mm" V 4380 4350 50  0001 C CNN
 F 3 "" H 4450 4350 50  0000 C CNN
@@
 P 5350 4850
 F 0 "R15" V 5430 4850 50  0000 C CNN
-F 1 "R" V 5350 4850 50  0000 C CNN
+F 1 "4.7K" V 5350 4850 50  0000 C CNN
 F 2 "Resistors_ThroughHole:Resistor_Horizontal_RM10mm" V 5280 4850 50  0001 C CNN
 F 3 "" H 5350 4850 50  0000 C CNN
@@
 P 5800 4350
 F 0 "R12" V 5880 4350 50  0000 C CNN
-F 1 "R" V 5800 4350 50  0000 C CNN
+F 1 "1K" V 5800 4350 50  0000 C CNN
 F 2 "Resistors_ThroughHole:Resistor_Horizontal_RM10mm" V 5730 4350 50  0001 C CNN
 F 3 "" H 5800 4350 50  0000 C CNN
@@
 P 6700 4850
 F 0 "R16" V 6780 4850 50  0000 C CNN
-F 1 "R" V 6700 4850 50  0000 C CNN
+F 1 "4.7K" V 6700 4850 50  0000 C CNN
 F 2 "Resistors_ThroughHole:Resistor_Horizontal_RM10mm" V 6630 4850 50  0001 C CNN
 F 3 "" H 6700 4850 50  0000 C CNN
